File: ecumodular.kicad_pcb (KiCad board)
At the start: 2 copper layers, 1 part, among them M1 Module-mega-mcu144-0.7

Commit message: 144mega
Other:
- board outline added: 237.6 x 130.5 mm
Changed lines of the file:
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@@
 		)
 	)
+	(gr_rect
+		(start 41.5 28)
+		(end 279.1 158.5)
+		(stroke
+			(width 0.05)
+			(type default)
+		)
+		(fill none)
+		(layer "Edge.Cuts")
+	)
 )
