File: ecumodular.kicad_pcb (KiCad board)
At the start: 2 copper layers, 237.6 x 130.5 mm, 1 part, among them M1 Module-mega-mcu144-0.7

Commit message: agregar
Parts:
- moved M1 75.1 mm to (44.4, 155.2)
Other:
- board size 237.6 x 130.5 mm -> 48.8 x 45.6 mm
Changed lines of the file:
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@@
 	(footprint "hellen-one-mega-mcu144-0.7:mega-mcu144"
 		(layer "F.Cu")
-		(at 48.999999 80.300007)
+		(at 44.374999 155.225003)
 		(property "Reference" "M1"
 			(at 43.2181 -40.093895 -90)
@@
 			(polygon
 				(pts
-					(xy 91.199998 80.200008) (xy 49.099998 80.200008) (xy 49.099998 40.300009) (xy 91.200001 40.300009)
+					(xy 86.574998 155.125004) (xy 44.474998 155.125004) (xy 44.474998 115.225005) (xy 86.575001 115.225005)
 				)
 			)
@@
 	)
 	(gr_rect
-		(start 41.5 28)
-		(end 279.1 158.5)
+		(start 41.5 112.9)
+		(end 90.3 158.5)
 		(stroke
 			(width 0.05)
